File: pcb/right/right.sch (KiCad schematic (older format))
At the start: 1 part

Commit message: Use basic symbol libraries
Connections:
- no-connect marks 3 -> 4
Changed lines of the file:
@@
 EESchema Schematic File Version 4
-LIBS:right-cache
 EELAYER 26 0
 EELAYER END
@@
 NoConn ~ 5600 4300
 $Comp
-L basic:+5V #PWR010
+L power:+5V #PWR010
 U 1 1 5A3F6A2D
 P 4800 4000
@@
 $EndComp
 $Comp
-L basic:GND #PWR011
+L power:GND #PWR011
 U 1 1 5A3F6A6E
 P 5800 4000
@@
 $EndComp
 $Comp
-L basic:PWR_FLAG #FLG04
+L power:PWR_FLAG #FLG04
 U 1 1 5A424761
 P 4800 4000
@@
 $EndComp
 $Comp
-L basic:PWR_FLAG #FLG02
+L power:PWR_FLAG #FLG02
 U 1 1 5A42418B
 P 5800 4000
@@
 Wire Wire Line
 	5200 3300 6100 3300
+NoConn ~ 4800 5100
 $EndSCHEMATC
