File: pcb/left/left.sch (KiCad schematic (older format))
At the start: 21 parts, among them CON1 AVR-ISP-6, J1 USB_OTG, J2 RJ11, SW1 SW_Push, U1 ATMEGA32U4-AU

Commit message: Update EEschema files for KiCad nightly
Parts:
- removed J2: RJ11, symbol RJ11
- added J?: RJ45, symbol Connector:RJ45
- 16MHz1: symbol Crystal_GND24 -> basic:Crystal_GND24
- C1, C10, C2, C3, C4, C5, C6, C7, C8, C9: symbol CP1_Small -> basic:CP1_Small
- CON1: symbol AVR-ISP-6 -> avr-isp-6:AVR-ISP-6
- J1: symbol USB_OTG -> usb_otg:USB_OTG
- R1, R2, R3, R4, R5: symbol R -> basic:R
- SW1: symbol SW_Push -> basic:SW_Push
- U1: symbol ATMEGA32U4-AU -> atmega32u4-au:ATMEGA32U4-AU
Connections:
- wire segments 70 -> 90
- no-connect marks 26 -> 28

Commit message: Use basic symbol libraries
Parts:
- removed CON1: AVR-ISP-6, AVR-ISP-6, symbol avr-isp-6:AVR-ISP-6
- added CON1: AVR-ISP-6, symbol atmel:AVR-ISP-6
- 16MHz1: symbol basic:Crystal_GND24 -> device:Crystal_GND24
- C1, C10, C2, C3, C4, C5, C6, C7, C8, C9: symbol basic:CP1_Small -> device:CP1_Small
- J1: symbol usb_otg:USB_OTG -> Connector:USB_OTG
- R1, R2, R3, R4, R5: symbol basic:R -> device:R
- SW1: symbol basic:SW_Push -> Switch:SW_Push
- U1: symbol atmega32u4-au:ATMEGA32U4-AU -> atmel:ATMEGA32U4-AU
Connections:
- wire segments 90 -> 83
Changed lines of the file:
@@
 EESchema Schematic File Version 4
-LIBS:left-cache
 EELAYER 26 0
 EELAYER END
@@
 $EndSheet
 $Comp
-L atmega32u4-au:ATMEGA32U4-AU U1
+L atmel:ATMEGA32U4-AU U1
 U 1 1 5A42392B
 P 4850 3650
@@
 $EndComp
 $Comp
-L basic:+5V #PWR01
+L power:+5V #PWR01
 U 1 1 5A4240F9
 P 2000 3300
@@
 $EndComp
 $Comp
-L basic:PWR_FLAG #FLG02
+L power:PWR_FLAG #FLG02
 U 1 1 5A42418B
 P 2000 3300
@@
 $EndComp
 $Comp
-L usb_otg:USB_OTG J1
+L Connector:USB_OTG J1
 U 1 1 5A42424B
 P 1500 3500
@@
 $EndComp
 $Comp
-L basic:R R1
+L device:R R1
 U 1 1 5A42447E
 P 3550 3450
@@
 $EndComp
 $Comp
-L basic:R R2
+L device:R R2
 U 1 1 5A4244E6
 P 3550 3550
@@
 $EndComp
 $Comp
-L basic:GND #PWR03
+L power:GND #PWR03
 U 1 1 5A42472F
 P 1800 4100
@@
 $EndComp
 $Comp
-L basic:PWR_FLAG #FLG04
+L power:PWR_FLAG #FLG04
 U 1 1 5A424761
 P 1800 4100
@@
 $EndComp
 $Comp
-L basic:GND #PWR05
+L power:GND #PWR05
 U 1 1 5A424952
 P 3600 4000
@@
 NoConn ~ 3700 4500
 $Comp
-L basic:Crystal_GND24 16MHz1
+L device:Crystal_GND24 16MHz1
 U 1 1 5A424E8A
 P 2700 2600
@@
 $EndComp
 $Comp
-L basic:CP1_Small C2
+L device:CP1_Small C2
 U 1 1 5A4251BA
 P 2900 2900
@@
 $EndComp
 $Comp
-L basic:CP1_Small C1
+L device:CP1_Small C1
 U 1 1 5A425245
 P 2500 2900
@@
 $EndComp
 $Comp
-L basic:GND #PWR06
+L power:GND #PWR06
 U 1 1 5A42529A
 P 2500 3000
@@
 $EndComp
 $Comp
-L basic:GND #PWR07
+L power:GND #PWR07
 U 1 1 5A4252C8
 P 2900 3000
@@
 $EndComp
 $Comp
-L basic:GND #PWR08
+L power:GND #PWR08
 U 1 1 5A425B6A
 P 2700 3000
@@
 $EndComp
 $Comp
-L basic:GND #PWR09
+L power:GND #PWR09
 U 1 1 5A425BA8
 P 2700 2400
@@
 NoConn ~ 9100 3900
 $Comp
-L basic:+5V #PWR010
+L power:+5V #PWR010
 U 1 1 5A3F6A2D
 P 8600 3700
@@
 $EndComp
 $Comp
-L basic:GND #PWR011
+L power:GND #PWR011
 U 1 1 5A3F6A6E
 P 9000 3700
@@
 NoConn ~ 5950 5000
 $Comp
-L basic:CP1_Small C4
+L device:CP1_Small C4
 U 1 1 5A3F6CF3
 P 2200 3000
@@
 $EndComp
 $Comp
-L basic:SW_Push SW1
+L Switch:SW_Push SW1
 U 1 1 5A3F7613
 P 3100 1750
@@
 $EndComp
 $Comp
-L basic:GND #PWR012
+L power:GND #PWR012
 U 1 1 5A3F97CA
 P 2900 1750
@@
 $EndComp
 $Comp
-L avr-isp-6:AVR-ISP-6 CON1
-U 1 1 5A404795
-P 7850 2500
-F 0 "CON1" H 7745 2740 50  0000 C CNN
-F 1 "AVR-ISP-6" H 7585 2270 50  0000 L BNN
-F 2 "AVR-ISP-6" V 7330 2540 50  0001 C CNN
-F 3 "" H 7825 2500 50  0001 C CNN
-	1    7850 2500
-	1    0    0    -1
-$EndComp
-$Comp
-L basic:GND #PWR013
+L power:GND #PWR013
 U 1 1 5A404967
-P 8300 2600
-F 0 "#PWR013" H 8300 2350 50  0001 C CNN
-F 1 "GND" H 8300 2450 50  0000 C CNN
-F 2 "" H 8300 2600 50  0001 C CNN
-F 3 "" H 8300 2600 50  0001 C CNN
-	1    8300 2600
-	1    0    0    -1
-$EndComp
-$Comp
-L basic:+5V #PWR014
+P 8200 2900
+F 0 "#PWR013" H 8200 2650 50  0001 C CNN
+F 1 "GND" H 8200 2750 50  0000 C CNN
+F 2 "" H 8200 2900 50  0001 C CNN
+F 3 "" H 8200 2900 50  0001 C CNN
+	1    8200 2900
+	0    -1   -1   0
+$EndComp
+$Comp
+L power:+5V #PWR014
 U 1 1 5A4049BA
-P 8300 2400
-F 0 "#PWR014" H 8300 2250 50  0001 C CNN
-F 1 "+5V" H 8300 2540 50  0000 C CNN
-F 2 "" H 8300 2400 50  0001 C CNN
-F 3 "" H 8300 2400 50  0001 C CNN
-	1    8300 2400
-	1    0    0    -1
-$EndComp
-$Comp
-L basic:GND #PWR015
+P 7300 2900
+F 0 "#PWR014" H 7300 2750 50  0001 C CNN
+F 1 "+5V" H 7300 3040 50  0000 C CNN
+F 2 "" H 7300 2900 50  0001 C CNN
+F 3 "" H 7300 2900 50  0001 C CNN
+	1    7300 2900
+	0    -1   -1   0
+$EndComp
+$Comp
+L power:GND #PWR015
 U 1 1 5A40AE67
 P 2200 2900
@@
 $EndComp
 $Comp
-L basic:CP1_Small C3
+L device:CP1_Small C3
 U 1 1 5A40B5F8
 P 3600 3900
@@
 $EndComp
 $Comp
-L basic:R R3
+L device:R R3
 U 1 1 5A40BF1D
 P 3500 1250
@@
 $EndComp
 $Comp
-L basic:+5V #PWR016
+L power:+5V #PWR016
 U 1 1 5A40C00D
 P 3500 1100
@@
 	5950 3400 7400 3400
 Wire Wire Line
-	7950 2400 8300 2400
-Wire Wire Line
-	7950 2600 8300 2600
-Wire Wire Line
-	8500 2500 7950 2500
-Wire Wire Line
-	5950 2300 7500 2300
-Wire Wire Line
-	7300 2500 7700 2500
-Wire Wire Line
-	5950 2400 7700 2400
-Wire Wire Line
-	7700 2600 7400 2600
-Wire Wire Line
-	7300 2200 7300 2500
-Wire Wire Line
-	5950 2200 7300 2200
-Wire Wire Line
-	7500 2300 7500 2100
-Wire Wire Line
-	7500 2100 8500 2100
-Wire Wire Line
-	8500 2100 8500 2500
-Wire Wire Line
 	3500 2100 3700 2100
 Wire Wire Line
@@
 	3600 3700 3700 3700
 $Comp
-L basic:GND #PWR017
+L power:GND #PWR017
 U 1 1 5A40C4CC
 P 4350 5350
@@
 Wire Wire Line
 	8700 1750 8700 3000
-Connection ~ 7400 1750
-Wire Wire Line
-	7400 2600 7400 1750
-$Comp
-L basic:+5V #PWR018
+$Comp
+L power:+5V #PWR018
 U 1 1 5A413885
 P 4750 900
@@
 $EndComp
 $Comp
-L basic:CP1_Small C8
+L device:CP1_Small C8
 U 1 1 5A41388B
 P 4950 1000
@@
 $EndComp
 $Comp
-L basic:GND #PWR019
+L power:GND #PWR019
 U 1 1 5A413892
 P 4950 900
@@
 Connection ~ 4750 1100
 $Comp
-L basic:+5V #PWR020
+L power:+5V #PWR020
 U 1 1 5A413905
 P 4550 900
@@
 $EndComp
 $Comp
-L basic:CP1_Small C7
+L device:CP1_Small C7
 U 1 1 5A41390B
 P 4350 1000
@@
 $EndComp
 $Comp
-L basic:GND #PWR021
+L power:GND #PWR021
 U 1 1 5A413912
 P 4350 900
@@
 $EndComp
 $Comp
-L basic:+5V #PWR022
+L power:+5V #PWR022
 U 1 1 5A4139BF
 P 4150 900
@@
 $EndComp
 $Comp
-L basic:CP1_Small C6
+L device:CP1_Small C6
 U 1 1 5A4139C5
 P 3950 1000
@@
 $EndComp
 $Comp
-L basic:GND #PWR023
+L power:GND #PWR023
 U 1 1 5A4139CB
 P 3950 900
@@
 Connection ~ 4150 1100
 $Comp
-L basic:+5V #PWR024
+L power:+5V #PWR024
 U 1 1 5A4142CF
 P 5150 900
@@
 $EndComp
 $Comp
-L basic:CP1_Small C9
+L device:CP1_Small C9
 U 1 1 5A4142D5
 P 5350 1000
@@
 $EndComp
 $Comp
-L basic:GND #PWR025
+L power:GND #PWR025
 U 1 1 5A4142DB
 P 5350 900
@@
 	5350 1100 5150 1100
 $Comp
-L basic:+5V #PWR026
+L power:+5V #PWR026
 U 1 1 5A414382
 P 5550 900
@@
 $EndComp
 $Comp
-L basic:CP1_Small C10
+L device:CP1_Small C10
 U 1 1 5A414388
 P 5750 1000
@@
 $EndComp
 $Comp
-L basic:GND #PWR027
+L power:GND #PWR027
 U 1 1 5A41438E
 P 5750 900
@@
 	4400 1500 4400 1850
 $Comp
-L basic:CP1_Small C5
+L device:CP1_Small C5
 U 1 1 5A4146BB
 P 3600 3150
@@
 $EndComp
 $Comp
-L basic:GND #PWR028
+L power:GND #PWR028
 U 1 1 5A4146C1
 P 3600 3050
@@
 	3400 3300 3600 3300
 $Comp
-L basic:+5V #PWR029
+L power:+5V #PWR029
 U 1 1 5A4148C9
 P 3400 3050
@@
 	3600 3300 3600 3250
 $Comp
-L basic:R R4
+L device:R R4
 U 1 1 5A489386
 P 7200 3650
@@
 $EndComp
 $Comp
-L basic:R R5
+L device:R R5
 U 1 1 5A489418
 P 7400 3650
@@
 	7400 3500 7400 3400
 $Comp
-L basic:+5V #PWR030
+L power:+5V #PWR030
 U 1 1 5A489589
 P 7200 3800
@@
 $EndComp
 $Comp
-L basic:+5V #PWR031
+L power:+5V #PWR031
 U 1 1 5A489652
 P 7400 3800
@@
 Wire Wire Line
 	3500 1750 3500 2100
-Wire Wire Line
-	3500 1750 7400 1750
-Wire Wire Line
-	7400 1750 8700 1750
 Wire Wire Line
 	4750 1100 4750 1850
@@
 Connection ~ 8800 3300
 NoConn ~ 8300 4700
+$Comp
+L atmel:AVR-ISP-6 CON1
+U 1 1 5A4C5D31
+P 7800 2800
+F 0 "CON1" V 7526 2850 50  0000 C CNN
+F 1 "AVR-ISP-6" V 7435 2850 50  0000 C CNN
+F 2 "" V 7550 2850 50  0001 C CNN
+F 3 "" H 6525 2250 50  0001 C CNN
+	1    7800 2800
+	0    -1   -1   0
+$EndComp
+Wire Wire Line
+	5950 2400 7600 2400
+Wire Wire Line
+	7700 2300 7700 2400
+Wire Wire Line
+	5950 2300 7700 2300
+Wire Wire Line
+	7800 2200 7800 2400
+Wire Wire Line
+	5950 2200 7800 2200
+Wire Wire Line
+	7900 2400 7900 1750
+Connection ~ 7900 1750
+Wire Wire Line
+	7900 1750 8700 1750
+Wire Wire Line
+	3500 1750 7900 1750
 $EndSCHEMATC

Commit message: Add TFT controller to schematic
Parts:
- added R6, R7, R8: 4.7K, symbol device:R
- added U2: ILI9341, symbol ili9341:ILI9341
- Y1: renamed from 16MHz1; value Crystal_GND24 -> 16MHz
- gave numbers to parts that had none: 1
Connections:
- net labels added: RESET, SCL, SDA, TFT_D0, TFT_D1, TFT_D2, TFT_D3, TFT_D4, TFT_D5, TFT_D6, TFT_D7, TFT_D[0..7], XTAL1, XTAL2
- wire segments 83 -> 109
- no-connect marks 28 -> 17
